Commit message: update for head

File: gazebo_simulation/camera/urdf/camera.urdf (robot description, URDF)
Before this commit: robot camera, 2 links, 1 joints
Joints:
- joint base_joint: origin xyz=0.0 0.0 1.2 rpy=0 0 0 -> xyz=0.0 0.0 1.5 rpy=0 0 0

File: gazebo_simulation/flov2tag/urdf/flov2tag.urdf (robot description, URDF)
Before this commit: robot flov2tag, 12 links, 11 joints
Joints:
- joint base_joint: origin xyz=0.0 0.0 1 rpy=0 0 0 -> xyz=0.0 0.0 0.1 rpy=0 0 0

File: gazebo_simulation/flov2withhead/urdf/flov2withhead.urdf (robot description, URDF)
Before this commit: robot flov2withhead, 12 links, 11 joints
Joints:
- joint l1: limit lower=-3.14 upper=3.14 effort=100 velocity=1 -> lower=-3.14 upper=3.14 effort=100 velocity=10
- joint l2: limit lower=-3.14 upper=3.14 effort=100 velocity=1 -> lower=-3.14 upper=3.14 effort=100 velocity=10
- joint l3: limit lower=-3.14 upper=3.14 effort=100 velocity=1 -> lower=-3.14 upper=3.14 effort=100 velocity=10; origin xyz=0.117 0 -0.00100000000000006 rpy=-1.5707963267949 0 -1.5707963267949 -> xyz=0.117 0 -0.00100000000000006 rpy=-1.57079632679491 0 -1.5707963267949
- joint l4: limit lower=-3.14 upper=3.14 effort=100 velocity=1 -> lower=-3.14 upper=3.14 effort=100 velocity=10
- joint r1: limit lower=-3.14 upper=3.14 effort=100 velocity=1 -> lower=-3.14 upper=3.14 effort=100 velocity=10
- joint r2: limit lower=-3.14 upper=3.14 effort=100 velocity=1 -> lower=-3.14 upper=3.14 effort=100 velocity=10
- joint r3: limit lower=-3.14 upper=3.14 effort=100 velocity=1 -> lower=-3.14 upper=3.14 effort=100 velocity=10
- joint r4: limit lower=-3.14 upper=3.14 effort=100 velocity=1 -> lower=-3.14 upper=3.14 effort=100 velocity=10

File: gazebo_simulation/test_moveit/config/gazebo_flov2tag.urdf (robot description, URDF)
Before this commit: robot flov2tag, 12 links, 11 joints
Joints:
- joint base_joint: origin xyz=0.0 0.0 0.0 rpy=0 0 0 -> xyz=0.0 0.0 1 rpy=0 0 0
