Commit message: Update URDF and launch files to reference new robot description package. Change mesh file paths from 'flov2withhead' to 'flov2_robot_description' for consistency. Modify camera launch configurations to use '/dev/video2' instead of '/dev/video0'. Enhance AprilTag detection script with updated camera parameters and improved logging. Adjust planning pipeline launch files to load configurations from the new package structure.

File: gazebo_simulation_and_control/flo_core/config/gazebo_flov2withhead.urdf (robot description, URDF)
Before this commit: robot flov2withhead, 12 links, 11 joints
Links:
- link base_link: geometry collision mesh filename=package://flov2_robot_description/meshes/base_link.STL; visual mesh filename=package://flov2_robot_description/meshes/base_link.STL
- link left_gripper: geometry collision mesh filename=package://flov2_robot_description/meshes/left_gripper.STL; visual mesh filename=package://flov2_robot_description/meshes/left_gripper.STL
- link left_low_arm: geometry collision mesh filename=package://flov2_robot_description/meshes/left_low_arm.STL; visual mesh filename=package://flov2_robot_description/meshes/left_low_arm.STL
- link left_low_joint: geometry collision mesh filename=package://flov2_robot_description/meshes/left_low_joint.STL; visual mesh filename=package://flov2_robot_description/meshes/left_low_joint.STL
- link left_up_arm: geometry collision mesh filename=package://flov2_robot_description/meshes/left_up_arm.STL; visual mesh filename=package://flov2_robot_description/meshes/left_up_arm.STL
- link left_up_joint: geometry collision mesh filename=package://flov2_robot_description/meshes/left_up_joint.STL; visual mesh filename=package://flov2_robot_description/meshes/left_up_joint.STL
- link right_gripper: geometry collision mesh filename=package://flov2_robot_description/meshes/right_gripper.STL; visual mesh filename=package://flov2_robot_description/meshes/right_gripper.STL
- link right_low_arm: geometry collision mesh filename=package://flov2_robot_description/meshes/right_low_arm.STL; visual mesh filename=package://flov2_robot_description/meshes/right_low_arm.STL
- link right_low_joint: geometry collision mesh filename=package://flov2_robot_description/meshes/right_low_joint.STL; visual mesh filename=package://flov2_robot_description/meshes/right_low_joint.STL
- link right_up_arm: geometry collision mesh filename=package://flov2_robot_description/meshes/right_up_arm.STL; visual mesh filename=package://flov2_robot_description/meshes/right_up_arm.STL
- link right_up_joint: geometry collision mesh filename=package://flov2_robot_description/meshes/right_up_joint.STL; visual mesh filename=package://flov2_robot_description/meshes/right_up_joint.STL

File: gazebo_simulation_and_control/flo_vision/urdf/flov2withhead.urdf (robot description, URDF)
Before this commit: robot flov2withhead, 7 links, 6 joints
Links:
- link base_link: geometry collision mesh filename=package://flov2_robot_description/meshes/base_link.STL; visual mesh filename=package://flov2_robot_description/meshes/base_link.STL
- link right_gripper: geometry collision mesh filename=package://flov2_robot_description/meshes/right_gripper.STL; visual mesh filename=package://flov2_robot_description/meshes/right_gripper.STL
- link right_low_arm: geometry collision mesh filename=package://flov2_robot_description/meshes/right_low_arm.STL; visual mesh filename=package://flov2_robot_description/meshes/right_low_arm.STL
- link right_low_joint: geometry collision mesh filename=package://flov2_robot_description/meshes/right_low_joint.STL; visual mesh filename=package://flov2_robot_description/meshes/right_low_joint.STL
- link right_up_arm: geometry collision mesh filename=package://flov2_robot_description/meshes/right_up_arm.STL; visual mesh filename=package://flov2_robot_description/meshes/right_up_arm.STL
- link right_up_joint: geometry collision mesh filename=package://flov2_robot_description/meshes/right_up_joint.STL; visual mesh filename=package://flov2_robot_description/meshes/right_up_joint.STL

File: gazebo_simulation_and_control/flov2_robot_description/urdf/flov2withhead.urdf (robot description, URDF)
Before this commit: robot flov2withhead, 12 links, 11 joints
Links:
- link base_link: geometry collision mesh filename=package://flov2_robot_description/meshes/base_link.STL; visual mesh filename=package://flov2_robot_description/meshes/base_link.STL
- link left_gripper: geometry collision mesh filename=package://flov2_robot_description/meshes/left_gripper.STL; visual mesh filename=package://flov2_robot_description/meshes/left_gripper.STL
- link left_low_arm: geometry collision mesh filename=package://flov2_robot_description/meshes/left_low_arm.STL; visual mesh filename=package://flov2_robot_description/meshes/left_low_arm.STL
- link left_low_joint: geometry collision mesh filename=package://flov2_robot_description/meshes/left_low_joint.STL; visual mesh filename=package://flov2_robot_description/meshes/left_low_joint.STL
- link left_up_arm: geometry collision mesh filename=package://flov2_robot_description/meshes/left_up_arm.STL; visual mesh filename=package://flov2_robot_description/meshes/left_up_arm.STL
- link left_up_joint: geometry collision mesh filename=package://flov2_robot_description/meshes/left_up_joint.STL; visual mesh filename=package://flov2_robot_description/meshes/left_up_joint.STL
- link right_gripper: geometry collision mesh filename=package://flov2_robot_description/meshes/right_gripper.STL; visual mesh filename=package://flov2_robot_description/meshes/right_gripper.STL
- link right_low_arm: geometry collision mesh filename=package://flov2_robot_description/meshes/right_low_arm.STL; visual mesh filename=package://flov2_robot_description/meshes/right_low_arm.STL
- link right_low_joint: geometry collision mesh filename=package://flov2_robot_description/meshes/right_low_joint.STL; visual mesh filename=package://flov2_robot_description/meshes/right_low_joint.STL
- link right_up_arm: geometry collision mesh filename=package://flov2_robot_description/meshes/right_up_arm.STL; visual mesh filename=package://flov2_robot_description/meshes/right_up_arm.STL
- link right_up_joint: geometry collision mesh filename=package://flov2_robot_description/meshes/right_up_joint.STL; visual mesh filename=package://flov2_robot_description/meshes/right_up_joint.STL
